File: board/board.kicad_pcb (KiCad board)
At the start: 2 copper layers, 21 x 13 mm, 1 part

Commit message: initial
Parts:
- added C1: 10uF, Capacitor_SMD:C_0603_1608Metric, F.Cu at (147.1, 100.1)
- added C2: 1uF, Capacitor_SMD:C_0603_1608Metric, F.Cu at (161.5, 93.2)
- added C3: 100nF, Capacitor_SMD:C_0603_1608Metric, F.Cu at (163.0, 93.2)
- added C4: 10nF, Capacitor_SMD:C_0603_1608Metric, F.Cu at (165.1, 94.5)
- added C5: 10nF, Capacitor_SMD:C_0603_1608Metric, F.Cu at (165.1, 97.5)
- added C6: 10nF, Capacitor_SMD:C_0603_1608Metric, F.Cu at (165.1, 100.6)
- added D1: NUP2105LT1G, Package_TO_SOT_SMD:SOT-23, F.Cu at (172.4, 97.6)
- added FB1: FerriteBead_Small, Inductor_SMD:L_0603_1608Metric, F.Cu at (147.1, 98.5)
- added FB2: BLM18BB471SN1D, Inductor_SMD:L_0603_1608Metric, F.Cu at (176.0, 96.6)
- added FB3: BLM18BB471SN1D, Inductor_SMD:L_0603_1608Metric, F.Cu at (176.0, 98.5)
- added J1: 002_SPI, on_edge:on_edge_2x05_device, F.Cu at (140.0, 96.5)
- added J2: 007_ADC, on_edge:on_edge_2x05_host, F.Cu at (185.0, 96.5)
- added R1: 1M, Resistor_SMD:R_0603_1608Metric, F.Cu at (169.5, 94.5)
- added R2: 1M, Resistor_SMD:R_0603_1608Metric, F.Cu at (169.5, 97.5)
- added R3: 1M, Resistor_SMD:R_0603_1608Metric, F.Cu at (169.5, 100.6)
- added U1: MAX31855KASA, Package_SO:SOIC-8_3.9x4.9mm_P1.27mm, F.Cu at (160.5, 97.6)
- moved LOGO1 2.81 mm to (152.8, 99.2)
Routing:
- net GND: track 0.00 -> 74.1 mm, vias 0 -> 6
- net +3.3V: track 0.00 -> 41.3 mm, vias 0 -> 1
- net +5V: track 0.00 -> 40.2 mm
- net /thermocouple/SCK: track 0.00 -> 22.3 mm
- net /thermocouple/VCC: track 0.00 -> 22.2 mm, vias 0 -> 2
- net /thermocouple/CS: track 0.00 -> 17.4 mm, vias 0 -> 1
- net /thermocouple/SO: track 0.00 -> 16.4 mm
- net Net-(C5-Pad2): track 0.00 -> 15.3 mm
- net Net-(C4-Pad2): track 0.00 -> 15.2 mm
- net /thermocouple/T+: track 0.00 -> 5.94 mm
- net /thermocouple/T-: track 0.00 -> 5.89 mm
Other:
- board size 21 x 13 mm -> 45 x 13 mm
- board text added: "osf.002"
- board text added: "osf.007"
- board text added: "osf.b016.v1.0"
